Commit message: fixed left right bug

File: urdf/srs-77dof.urdf (robot description, URDF)
Before this commit: robot srs-77dof, 15 links, 14 joints
Links:
- added link left_tcp
- added link right_tcp
- link link-l1: mass 2.89937170911004 -> 2.8994; geometry collision mesh filename=package://srs-77dof/meshes/link-r1.STL; visual mesh filename=package://srs-77dof/meshes/link-r1.STL
- link link-l2: mass 4.49590564030825 -> 4.4959; geometry collision mesh filename=package://srs-77dof/meshes/link-r2.STL; visual mesh filename=package://srs-77dof/meshes/link-r2.STL
- link link-l3: mass 1.50985052864978 -> 1.50987241060898; geometry collision mesh filename=package://srs-77dof/meshes/link-r3.STL; visual mesh filename=package://srs-77dof/meshes/link-r3.STL
- link link-l4: mass 2.0375685441998 -> 2.0376; geometry collision mesh filename=package://srs-77dof/meshes/link-r4.STL; visual mesh filename=package://srs-77dof/meshes/link-r4.STL
- link link-l5: mass 1.50985052900885 -> 1.5099; geometry collision mesh filename=package://srs-77dof/meshes/link-r5.STL; visual mesh filename=package://srs-77dof/meshes/link-r5.STL
- link link-l6: mass 1.77721693197758 -> 1.7772; geometry collision mesh filename=package://srs-77dof/meshes/link-r6.STL; visual mesh filename=package://srs-77dof/meshes/link-r6.STL
- link link-l7: mass 0.30505900233751 -> 0.30506; geometry collision mesh filename=package://srs-77dof/meshes/link-r7.STL; visual mesh filename=package://srs-77dof/meshes/link-r7.STL
- link link-r1: mass 2.8994 -> 2.89937170911004; geometry collision mesh filename=package://srs-77dof/meshes/link-l1.STL; visual mesh filename=package://srs-77dof/meshes/link-l1.STL
- link link-r2: mass 4.4959 -> 4.49590564030825; geometry collision mesh filename=package://srs-77dof/meshes/link-l2.STL; visual mesh filename=package://srs-77dof/meshes/link-l2.STL
- link link-r3: mass 1.50987241060898 -> 1.50985052864978; geometry collision mesh filename=package://srs-77dof/meshes/link-l3.STL; visual mesh filename=package://srs-77dof/meshes/link-l3.STL
- link link-r4: mass 2.0376 -> 2.0375685441998; geometry collision mesh filename=package://srs-77dof/meshes/link-l4.STL; visual mesh filename=package://srs-77dof/meshes/link-l4.STL
- link link-r5: mass 1.5099 -> 1.50985052900885; geometry collision mesh filename=package://srs-77dof/meshes/link-l5.STL; visual mesh filename=package://srs-77dof/meshes/link-l5.STL
- link link-r6: mass 1.7772 -> 1.77721693197758; geometry collision mesh filename=package://srs-77dof/meshes/link-l6.STL; visual mesh filename=package://srs-77dof/meshes/link-l6.STL
- link link-r7: mass 0.30506 -> 0.30505900233751; geometry collision mesh filename=package://srs-77dof/meshes/link-l7.STL; visual mesh filename=package://srs-77dof/meshes/link-l7.STL
Joints:
- added joint fix_tcp_l: type fixed, parent link-l7, child left_tcp, origin xyz=0 -0.2 0 rpy=3.14 0 0
- added joint fix_tcp_r: type fixed, parent link-r7, child right_tcp, origin xyz=0.2 0 0 rpy=0 3.14 -1.5708
- joint joint-l1: axis -1 0 0 -> 0 0 -1; origin xyz=-0.3325 0 0.53254 rpy=-1.5708 0 -3.1416 -> xyz=0.3325 0 0.53254 rpy=3.14 -1.5708 0
- joint joint-l2: axis 1 0 0 -> 0 0 1
- joint joint-l3: axis 1 0 0 -> 0 0 1; origin xyz=0 0 0 rpy=-1.5708 -1.5708 0 -> xyz=0 0 0 rpy=1.5708 1.5708 0
- joint joint-l4: axis 0 0 1 -> 0 0 -1; origin xyz=0.2651 -4E-05 0 rpy=0 0 0 -> xyz=4E-05 0 0.2651 rpy=1.5708 1.5708 0
- joint joint-l5: origin xyz=0 0.2653 0.00015 rpy=-1.5708 0 0 -> xyz=0 -0.2653 0 rpy=1.5708 0 0
- joint joint-l6: origin xyz=0 0 0 rpy=1.5708 -1.5708 0 -> xyz=0 0 0 rpy=1.5708 1.5708 0
- joint joint-l7: origin xyz=0 0 0 rpy=1.5708 0 0 -> xyz=0 0 0 rpy=1.5708 1.5708 0
- joint joint-r1: axis 0 0 -1 -> -1 0 0; origin xyz=0.3325 0 0.53254 rpy=3.14 -1.5708 0 -> xyz=-0.3325 0 0.53254 rpy=-1.5708 0 -3.1416
- joint joint-r2: axis 0 0 1 -> 1 0 0
- joint joint-r3: axis 0 0 1 -> 1 0 0; origin xyz=0 0 0 rpy=1.5708 1.5708 0 -> xyz=0 0 0 rpy=-1.5708 -1.5708 0
- joint joint-r4: axis 0 0 -1 -> 0 0 1; origin xyz=4E-05 0 0.2651 rpy=1.5708 1.5708 0 -> xyz=0.2651 0 0 rpy=0 0 0
- joint joint-r5: origin xyz=0 -0.2653 -0.00015 rpy=1.5708 0 0 -> xyz=0 0.2653 0 rpy=-1.5708 0 0
- joint joint-r6: origin xyz=0 0 0 rpy=1.5708 1.5708 0 -> xyz=0 0 0 rpy=1.5708 -1.5708 0
- joint joint-r7: origin xyz=0 0 0 rpy=1.5708 1.5708 0 -> xyz=0 0 0 rpy=1.5708 0 0
